File: line-sensor-v1.kicad_pcb (KiCad board)
At the start: 2 copper layers, 20 parts

Commit message: commit
Parts:
- moved U7 173.9 mm to (223.5, 101.6)
- moved U9 170.2 mm to (241.3, 83.8)
- moved U15 160.6 mm to (222.2, 77.5)
- moved U16 160.5 mm to (222.2, 79.5)
- moved U17 160.4 mm to (222.2, 81.5)
- moved U18 160.3 mm to (222.2, 83.5)
- moved U19 160.3 mm to (222.2, 85.5)
- moved U10 154.7 mm to (204.5, 91.4)
- moved U11 154.7 mm to (204.5, 109.2)
- moved U12 154.7 mm to (222.2, 109.2)
- moved U13 154.7 mm to (240.0, 109.2)
- moved U14 154.7 mm to (240.0, 91.4)
- moved U4 154.6 mm to (229.9, 91.4)
- moved U8 153.4 mm to (241.3, 101.6)
- moved U5 152.4 mm to (205.7, 83.8)
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Routing:
- net Net-(U1-4): track 0.00 -> 192.5 mm
- net Net-(U1-3V3): track 0.64 -> 172.6 mm
- net Net-(U1-34): track 0.00 -> 118.3 mm
- net Net-(U1-35): track 0.00 -> 103.5 mm
- net Net-(U4-C): track 0.00 -> 96.2 mm
- net Net-(U3-C): track 0.00 -> 80.6 mm
- net Net-(U2-C): track 0.00 -> 79.1 mm
- net Net-(U1-12): track 0.00 -> 46.5 mm
- net Net-(U1-15): track 1.41 -> 0.00 mm

Commit message: finished pcb
Parts:
- moved U1 86.4 mm to (141.0, 76.2)
- moved U12 86.4 mm to (139.7, 134.6)
- moved U13 86.4 mm to (157.5, 134.6)
- moved U14 86.4 mm to (157.5, 116.8)
- moved U15 86.4 mm to (139.7, 102.9)
- moved U16 86.4 mm to (139.7, 104.9)
- moved U17 86.4 mm to (139.7, 106.9)
- moved U18 86.4 mm to (139.7, 108.9)
- moved U19 86.4 mm to (139.7, 110.9)
- moved U20 86.4 mm to (139.7, 82.5)
- moved U3 86.4 mm to (139.7, 116.8)
- moved U4 86.4 mm to (147.3, 116.8)
- moved U5 86.4 mm to (123.2, 109.2)
- moved U6 86.4 mm to (123.2, 127.0)
- moved U7 86.4 mm to (141.0, 127.0)
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Routing:
- net Net-(U1-26): track 0.00 -> 94.8 mm
- net Net-(U1-15): track 0.00 -> 77.3 mm
- net Net-(U2-E): track 0.00 -> 67.2 mm
- net Net-(U1-25): track 0.00 -> 66.0 mm
- net Net-(U1-32): track 0.00 -> 51.9 mm
- net Net-(U1-Pad22): track 0.00 -> 27.9 mm
- net Net-(U1-5V): track 0.00 -> 24.3 mm
- net Net-(U1-21): track 0.00 -> 22.1 mm
- net Net-(U1-4): track 192.5 -> 200.3 mm
Other:
- board outline added: 50.8 x 88.9 mm
